Commit message: [ROS_robot] some fixes, many troubles with frictions

File: my_super_car/my_super_car_description/urdf/model.urdf.xacro (robot description, xacro)
@@ -3,11 +3,12 @@
   <xacro:property name="wheel_width" value="0.03" />
   <xacro:property name="wheel_radius" value="0.04" />
-  <xacro:property name="wheel_mass" value="0.3" />
+  <xacro:property name="wheel_mass" value="0.056" />
   <xacro:property name="wheel_chassis_bias" value="${wheel_width/2}" />
   <xacro:property name="chassis_mass" value="3.7" />
   <xacro:property name="chassis_length" value="0.485" />
   <xacro:property name="chassis_width" value="0.227" />
-  <xacro:property name="chassis_height" value="0.01" />
+  <xacro:property name="chassis_height" value="0.05" />
   <xacro:property name="wheelbase" value="0.3" />
+  <xacro:property name="lidar_mass" value="0.1" />
   <!-- https://github.com/jbpassot/ackermann_vehicle/blob/master/ackermann_vehicle_description/urdf/em_3905.urdf.xacro -->
   <xacro:property name="degrees_45" value="0.785398163"/>
@@ -74,8 +75,8 @@
       <mu1>1.2</mu1>
       <mu2>1.05</mu2>
-      <kp>10000000</kp>
-      <kd>1</kd>
-      <minDepth>0.01</minDepth>
-      <maxVel>10.0</maxVel>
+      <!-- <kp>10000000</kp> -->
+      <!-- <kd>1</kd>  -->
+      <!-- <minDepth>0.01</minDepth> -->
+      <!-- <maxVel>10.0</maxVel>  -->
       <material>Gazebo/Black</material>
     </gazebo>
@@ -89,5 +90,5 @@
       <axis xyz="0 0 -1"/>
     </joint>
-<!--     <transmission name="${name}_rotate_trans">
+    <transmission name="${name}_rotate_trans">
       <type>transmission_interface/SimpleTransmission</type>
       <joint name="${name}_rotate_joint">
@@ -97,5 +98,5 @@
         <mechanicalReduction>1</mechanicalReduction>
       </actuator>
-    </transmission> -->
+    </transmission>
   </xacro:macro>
   <xacro:macro name="steering_wheel" params="name base_name xyz ref">
@@ -177,10 +178,10 @@
   <xacro:steering_wheel name="left_steer_wheel" base_name="base_link" xyz="${wheelbase/2} ${chassis_width/2} 0" ref="1" />
  -->
-  <xacro:steering_wheel name="right_steer_wheel" base_name="base_link" xyz="${wheelbase/2} ${-(chassis_width/2 + wheel_chassis_bias)} 0" ref="-1" />
-  <xacro:steering_wheel name="left_steer_wheel" base_name="base_link" xyz="${wheelbase/2} ${(chassis_width/2 + wheel_chassis_bias)} 0" ref="1" />
+  <xacro:steering_wheel name="right_steer_wheel" base_name="base_link" xyz="${wheelbase/2} ${-(chassis_width/2 + wheel_chassis_bias)} ${-chassis_height/2}" ref="-1" />
+  <xacro:steering_wheel name="left_steer_wheel" base_name="base_link" xyz="${wheelbase/2} ${(chassis_width/2 + wheel_chassis_bias)} ${-chassis_height/2}" ref="1" />
   <xacro:traveling_wheel name="right_travel_wheel" base_name="base_link"
-                         xyz="${-wheelbase/2} ${-(chassis_width/2 + wheel_chassis_bias)} 0" />
+                         xyz="${-wheelbase/2} ${-(chassis_width/2 + wheel_chassis_bias)} ${-chassis_height/2}" />
   <xacro:traveling_wheel name="left_travel_wheel" base_name="base_link"
-                         xyz="${-wheelbase/2} ${(chassis_width/2 + wheel_chassis_bias)} 0" />
+                         xyz="${-wheelbase/2} ${(chassis_width/2 + wheel_chassis_bias)} ${-chassis_height/2}" />
   <!-- Gazebo plugin for ROS Control -->
   <gazebo>
@@ -189,3 +190,60 @@
     </plugin>
   </gazebo>
+  <xacro:property name="lidar_height" value="0.04"/>
+  <xacro:property name="lidar_radius" value="0.04"/>
+  <link name="hokuyo_link">
+    <xacro:solid_cylinder_inertial
+        r="${lidar_radius}" h="${lidar_height}"
+        mass="${lidar_mass}" >
+      <origin xyz="0 0 0" rpy="0 0 0" />
+    </xacro:solid_cylinder_inertial>
+    <collision>
+      <origin xyz="0 0 0" rpy="0 0 0" />
+      <geometry>
+        <cylinder length="${lidar_height}" radius="${lidar_radius}"/>
+      </geometry>
+    </collision>
+    <visual>
+      <origin xyz="0 0 0" rpy="0 0 0" />
+      <geometry>
+        <cylinder length="${lidar_height}" radius="${lidar_radius}"/>
+      </geometry>
+    </visual>
+  </link>
+  <joint name="hokuyo_joint" type="fixed">
+    <child link="hokuyo_link" />
+    <parent link="base_link" />
+    <origin xyz="0 0 ${chassis_height/2 + lidar_height/2}" />
+  </joint>
+  <gazebo reference="hokuyo_link">
+    <material>Gazebo/Black</material>
+    <sensor type="gpu_ray" name="head_hokuyo_sensor">
+      <visualize>true</visualize>
+      <update_rate>10</update_rate>
+      <ray>
+        <scan>
+          <horizontal>
+            <samples>360</samples>
+            <resolution>1</resolution>
+            <min_angle>-1.570796</min_angle>
+            <max_angle>1.570796</max_angle>
+          </horizontal>
+        </scan>
+        <range>
+          <min>0.10</min>
+          <max>10.0</max>
+          <resolution>0.01</resolution>
+        </range>
+        <noise>
+          <type>gaussian</type>
+          <mean>0.0</mean>
+          <stddev>0.01</stddev>
+        </noise>
+      </ray>
+      <plugin name="gazebo_ros_head_hokuyo_controller" filename="libgazebo_ros_gpu_laser.so">
+        <topicName>scan</topicName>
+        <frameName>hokuyo_link</frameName>
+      </plugin>
+    </sensor>
+  </gazebo>
 </robot>
